File: RaspberryPiHat/raspberry_pi_hat.sch (KiCad schematic (older format))
At the start: 11 parts, among them J1 CONN_2x20_FEM_100PITCH_635INS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, U1 CAT24C32

Commit message: rework done
Parts:
- removed C1: 100nF_CER_0603_50V, Capacitor_SMD:C_0603_1608Metric_Pad1.05x0.95mm_HandSolder, symbol JB_Cap_Smd_50v:100nF_CER_0603_50V
- removed J1: CONN_2x20_FEM_100PITCH_635INS_280POST, JB_Header_100mils:ESQ-120-34-G-D, symbol JB_Header_100mils:CONN_2x20_FEM_100PITCH_635INS_280POST
- removed JP1: Solder_Jumper_1.3MM, Jumper:SolderJumper-2_P1.3mm_Open_RoundedPad1.0x1.5mm, symbol JB_Jumper:Solder_Jumper_1.3MM
- removed MH1, MH2, MH3, MH4: MH-NPLTD-M2.5, MountingHole:MountingHole_2.7mm_M2.5_DIN965, symbol JB_Mechanical:MH-NPLTD-M2.5
- removed R1: 1K_0603_100MW, Resistor_SMD:R_0603_1608Metric_Pad1.05x0.95mm_HandSolder, symbol JB_Res_Smd_0w100:1K_0603_100MW
- removed R2, R3: 3K9_0603_100MW, Resistor_SMD:R_0603_1608Metric_Pad1.05x0.95mm_HandSolder, symbol JB_Res_Smd_0w100:3K9_0603_100MW
- removed U1: CAT24C32, Package_SO:SOIC-8_3.9x4.9mm_P1.27mm, symbol JB_Memory:CAT24C32
- added C1: 100nF_CER_0603_50V, Capacitor_SMD:C_0603_1608Metric_Pad1.05x0.95mm_HandSolder, symbol ENYA_Cap_Smd_50V:100nF_CER_0603_50V
- added J1: CONN_2x20_FEM_100PITCH_635INS_280POST, ENYA_Header_100mils:ESQ-120-34-G-D, symbol ENYA_Header_100mils:CONN_2x20_FEM_100PITCH_635INS_280POST
- added JP1: Solder_Jumper_1.3MM, Jumper:SolderJumper-2_P1.3mm_Open_RoundedPad1.0x1.5mm, symbol ENYA_Jumper:Solder_Jumper_1.3MM
- added MH1, MH2, MH3, MH4: MH-NPLTD-M2.5, MountingHole:MountingHole_2.7mm_M2.5_DIN965, symbol ENYA_Mechanical:MH-NPLTD-M2.5
- added R1: 1K_0603_100MW, Resistor_SMD:R_0603_1608Metric_Pad1.05x0.95mm_HandSolder, symbol ENYA_Res_Smd_100mW:1K_0603_100MW
- added R2, R3: 3K9_0603_100MW, Resistor_SMD:R_0603_1608Metric_Pad1.05x0.95mm_HandSolder, symbol ENYA_Res_Smd_100mW:3K9_0603_100MW
- added U1: CAT24C32, Package_SO:SOIC-8_3.9x4.9mm_P1.27mm, symbol ENYA_Memory:CAT24C32
Connections:
- net +3V3: now also C1.1, J1.1 (Pin_1), J1.17 (Pin_17), R1.1, R2.1, R3.1, U1.8 (VCC)
- net +5V: now also J1.2 (Pin_2), J1.4 (Pin_4)
- net GND: now also C1.2, J1.14 (Pin_14), J1.20 (Pin_20), J1.25 (Pin_25), J1.30 (Pin_30), J1.34 (Pin_34), J1.39 (Pin_39), J1.6 (Pin_6), J1.9 (Pin_9), JP1.2, U1.1 (A0), U1.2 (A1), U1.3 (A2), U1.4 (GND)
- net ID_SCL: now also J1.28 (Pin_28), R3.2, U1.6 (SCL)
- net ID_SDA: now also J1.27 (Pin_27), R2.2, U1.5 (SDA)
- new net: JP1.1, R1.2, U1.7 (WP)
