File: RaspberryPiHat/raspberry_pi_hat.sch (KiCad schematic (older format))
At the start: 11 parts, among them J1 CONN_2x20_FEM_100PITCH_635INS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, U1 CAT24C32

Commit message: Correcting typo on pi gpio connector signals
Other:
- note added: "GPIO15/RXD0"
- note removed: "GPIO15/TXD0"
Changed lines of the file:
@@
 GPIO14/TXD0
 Text Notes 3200 1600 0    50   ~ 0
-GPIO15/TXD0
+GPIO15/RXD0
 Text Notes 3200 1700 0    50   ~ 0
 GPIO18/GEN1

Commit message: updating project templates
Parts:
- removed J1: CONN_2x20_FEM_100PITCH_635INS_280POST, ENYA_Header_100mils:ESQ-120-34-G-D, symbol ENYA_Header_100mils:CONN_2x20_FEM_100PITCH_635INS_280POST
- added J1: CONN_2x20_FEM_100PITCH_335INS_126POST, ENYA_Header_100mils:PPTC202LFBN-RC, symbol ENYA_Header_100mils:CONN_2x20_FEM_100PITCH_335INS_126POST
Connections:
- net +3V3: now also J1.1 (Pin_1), J1.17 (Pin_17)
- net +5V: now also J1.2 (Pin_2), J1.4 (Pin_4)
- net GND: now also J1.14 (Pin_14), J1.20 (Pin_20), J1.25 (Pin_25), J1.30 (Pin_30), J1.34 (Pin_34), J1.39 (Pin_39), J1.6 (Pin_6), J1.9 (Pin_9)
- net ID_SCL: now also J1.28 (Pin_28)
- net ID_SDA: now also J1.27 (Pin_27)
Changed lines of the file:
@@
-$EndComp
-$Comp
-L ENYA_Header_100mils:CONN_2x20_FEM_100PITCH_635INS_280POST J1
-U 1 1 5EA72C40
-P 2700 2100
-F 0 "J1" H 2700 3125 50  0000 C CNN
-F 1 "CONN_2x20_FEM_100PITCH_635INS_280POST" H 2700 975 50  0001 C CNN
-F 2 "ENYA_Header_100mils:ESQ-120-34-G-D" H 2700 825 50  0001 C CNN
-F 3 "L:\\JudeBake\\Datasheet\\Header\\esq-1xx-xx-x-x-xxx-xx-x-xx-mkt.pdf" H 2700 750 50  0001 C CNN
-F 4 "Samtec" H 2700 2100 50  0001 C CNN "Manufacturer"
-F 5 "ESQ-120-34-G-D" H 2700 2100 50  0001 C CNN "Manufacturer Part Number"
-F 6 "SAM9319-ND" H 2700 2100 50  0001 C CNN "Digi-Key Part Number"
-	1    2700 2100
-	1    0    0    -1
 $EndComp
 $Comp
@@
 	1    0    0    -1
 $EndComp
+$Comp
+L ENYA_Header_100mils:CONN_2x20_FEM_100PITCH_335INS_126POST J1
+U 1 1 602DC295
+P 2700 2100
+F 0 "J1" H 2700 3125 50  0000 C CNN
+F 1 "CONN_2x20_FEM_100PITCH_335INS_126POST" H 2700 975 50  0001 C CNN
+F 2 "ENYA_Header_100mils:PPTC202LFBN-RC" H 2700 825 50  0001 C CNN
+F 3 "https://media.digikey.com/pdf/Data%20Sheets/Sullins%20PDFs/Female_Headers.100_DS.pdf" H 2700 750 50  0001 C CNN
+F 4 "Sullins Connector Solutions" H 2700 2100 50  0001 C CNN "Manufacturer"
+F 5 "PPTC202LFBN-RC" H 2700 2100 50  0001 C CNN "Manufacturer Part Number"
+F 6 "S6104-ND" H 2700 2100 50  0001 C CNN "Digi-Key Part Number"
+	1    2700 2100
+	1    0    0    -1
+$EndComp
