File: GeneralProject/general_project.kicad_pcb (KiCad board)
At the start: 2 copper layers, 0 parts

Commit message: migating to kicad 6
Other:
- net class Default removed
- net class PWR removed
- net class SIGNAL removed
Changed lines of the file:
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@@
-(kicad_pcb (version 20171130) (host pcbnew "(5.1.5)-3")
+(kicad_pcb (version 20211014) (generator pcbnew)
   (general
     (thickness 1.6)
-    (drawings 0)
-    (tracks 0)
-    (zones 0)
-    (modules 0)
-    (nets 1)
   )
-  (page USLedger)
+  (paper "USLedger")
   (layers
-    (0 F.Cu signal)
-    (31 B.Cu signal)
-    (32 B.Adhes user)
-    (33 F.Adhes user)
-    (34 B.Paste user)
-    (35 F.Paste user)
-    (36 B.SilkS user)
-    (37 F.SilkS user)
-    (38 B.Mask user)
-    (39 F.Mask user)
-    (40 Dwgs.User user)
-    (41 Cmts.User user)
-    (42 Eco1.User user)
-    (43 Eco2.User user)
-    (44 Edge.Cuts user)
-    (45 Margin user)
-    (46 B.CrtYd user)
-    (47 F.CrtYd user)
-    (48 B.Fab user)
-    (49 F.Fab user)
+    (0 "F.Cu" signal)
+    (31 "B.Cu" signal)
+    (32 "B.Adhes" user "B.Adhesive")
+    (33 "F.Adhes" user "F.Adhesive")
+    (34 "B.Paste" user)
+    (35 "F.Paste" user)
+    (36 "B.SilkS" user "B.Silkscreen")
+    (37 "F.SilkS" user "F.Silkscreen")
+    (38 "B.Mask" user)
+    (39 "F.Mask" user)
+    (40 "Dwgs.User" user "User.Drawings")
+    (41 "Cmts.User" user "User.Comments")
+    (42 "Eco1.User" user "User.Eco1")
+    (43 "Eco2.User" user "User.Eco2")
+    (44 "Edge.Cuts" user)
+    (45 "Margin" user)
+    (46 "B.CrtYd" user "B.Courtyard")
+    (47 "F.CrtYd" user "F.Courtyard")
+    (48 "B.Fab" user)
+    (49 "F.Fab" user)
   )
   (setup
-    (last_trace_width 0.1524)
-    (user_trace_width 0.1524)
-    (user_trace_width 0.254)
-    (user_trace_width 0.381)
-    (user_trace_width 0.508)
-    (user_trace_width 0.635)
-    (user_trace_width 1.27)
-    (trace_clearance 0.1524)
-    (zone_clearance 0.508)
-    (zone_45_only no)
-    (trace_min 0.1524)
-    (via_size 0.508)
-    (via_drill 0.254)
-    (via_min_size 0.508)
-    (via_min_drill 0.254)
-    (user_via 0.508 0.254)
-    (user_via 0.762 0.381)
-    (user_via 1.27 0.635)
-    (uvia_size 0.3)
-    (uvia_drill 0.1)
-    (uvias_allowed no)
-    (uvia_min_size 0.2)
-    (uvia_min_drill 0.1)
-    (edge_width 0.05)
-    (segment_width 0.2)
-    (pcb_text_width 0.3)
-    (pcb_text_size 1.5 1.5)
-    (mod_edge_width 0.12)
-    (mod_text_size 1 1)
-    (mod_text_width 0.15)
-    (pad_size 1.524 1.524)
-    (pad_drill 0.762)
     (pad_to_mask_clearance 0.051)
     (solder_mask_min_width 0.25)
-    (aux_axis_origin 0 0)
-    (visible_elements 7FFFFFFF)
     (pcbplotparams
-      (layerselection 0x010fc_ffffffff)
+      (layerselection 0x00010fc_ffffffff)
+      (disableapertmacros false)
       (usegerberextensions false)
       (usegerberattributes false)
       (usegerberadvancedattributes false)
       (creategerberjobfile false)
+      (svguseinch false)
+      (svgprecision 6)
       (excludeedgelayer true)
-      (linewidth 0.100000)
       (plotframeref false)
       (viasonmask false)
@@
       (hpglpenspeed 20)
       (hpglpendiameter 15.000000)
+      (dxfpolygonmode true)
+      (dxfimperialunits true)
+      (dxfusepcbnewfont true)
       (psnegative false)
       (psa4output false)
@@
       (plotvalue true)
       (plotinvisibletext false)
-      (padsonsilk false)
+      (sketchpadsonfab false)
       (subtractmaskfromsilk false)
       (outputformat 1)
@@
       (drillshape 1)
       (scaleselection 1)
-      (outputdirectory ""))
+      (outputdirectory "")
+    )
   )
   (net 0 "")
-  (net_class Default "This is the default net class."
-    (clearance 0.1524)
-    (trace_width 0.1524)
-    (via_dia 0.508)
-    (via_drill 0.254)
-    (uvia_dia 0.3)
-    (uvia_drill 0.1)
-  )
-  (net_class PWR ""
-    (clearance 0.1524)
-    (trace_width 0.1524)
-    (via_dia 0.508)
-    (via_drill 0.254)
-    (uvia_dia 0.3)
-    (uvia_drill 0.1)
-  )
-  (net_class SIGNAL ""
-    (clearance 0.1524)
-    (trace_width 0.1524)
-    (via_dia 0.508)
-    (via_drill 0.254)
-    (uvia_dia 0.3)
-    (uvia_drill 0.1)
-  )
 )
